Commit message: add pcd_proj_node

File: src/bring_up/urdf/sensor_suite.urdf.xacro (robot description, xacro)
@@ -8,5 +8,5 @@
   <link name="radar" />
   <joint name="base_joint" type="fixed">
-    <origin xyz="0 0 0" rpy="0 0 0" />
+    <origin xyz="0 0 0" rpy="0 0 ${-pi}" />
     <parent link="base_link" />
     <child link="os_lidar" />

Commit message: update projection

File: src/bring_up/urdf/sensor_suite.urdf.xacro (robot description, xacro)
@@ -2,13 +2,13 @@
 <robot name="sensor_suite"
   xmlns:xacro="http://ros.org/wiki/xacro">
+  <link name="os_lidar" />
   <link name="base_link" />
-  <link name="os_lidar" />
   <link name="cam_rgb" />
   <link name="cam_thermal" />
   <link name="radar" />
   <joint name="base_joint" type="fixed">
-    <origin xyz="0 0 0" rpy="0 0 ${-pi}" />
-    <parent link="base_link" />
-    <child link="os_lidar" />
+    <origin xyz="0 0 0" rpy="0 0 ${pi}" />
+    <parent link="os_lidar" />
+    <child link="base_link" />
   </joint>
   <joint name="cam_rgb_joint" type="fixed">

Commit message: update urdf

File: src/bring_up/urdf/sensor_suite.urdf.xacro (robot description, xacro)
@@ -2,13 +2,13 @@
 <robot name="sensor_suite"
   xmlns:xacro="http://ros.org/wiki/xacro">
+  <link name="base_link" />
   <link name="os_lidar" />
-  <link name="base_link" />
   <link name="cam_rgb" />
   <link name="cam_thermal" />
   <link name="radar" />
   <joint name="base_joint" type="fixed">
-    <origin xyz="0 0 0" rpy="0 0 ${pi}" />
-    <parent link="os_lidar" />
-    <child link="base_link" />
+    <origin xyz="0 0 0" rpy="0 0 ${-pi}" />
+    <parent link="base_link" />
+    <child link="os_lidar" />
   </joint>
   <joint name="cam_rgb_joint" type="fixed">
